Commit message: docs(sim): 以 scene.xml 为准对齐查看器模型（URDF 重建 + 连接件 + 去夹爪）
问题：docs/viewer/robot.urdf 原是"官方 piper_description URDF + 手"的拼装，与权威 MJCF
（sim/piper_linker/scene.xml）不一致：link3 起链路世界位置偏差 ~10mm（实测最大 11.2mm）、
8 处关节限位不同、link6 视觉用的是含夹爪的完整 link6.stl、且缺少灵巧手连接件 adapter。

做法：新增 sim/piper_linker/tools/sync_viewer_urdf.py，从 MJCF 生成查看器 URDF（可复现、可 --verify）：
- 关节 origin 直接取 MJCF body 的 pos/quat（→ URDF rpy）、轴取 MJCF axis、限位取 MJCF range
  （joint1 ±2.618、joint3 −2.697、joint4 ±1.832、joint6 ±3.14、thumb_ip 1.3282、各 dip 1.424 等随之一致）
- 视觉网格取 MJCF class=visual 的 geom 与其 quat：link6 → link6_trimmed（+ 连接件 adapter）；
  手基座仍挂在 link6 下 0.0175m（fixed lh_adapter_joint）
- link1~link5 的 MJCF 用官方"分片网格"（link2 有 32 片），与官方单文件 STL 逐点等价
  （包围盒 max 差 0.00mm，脚本内置该结论注释），故沿用单文件以省体积
- 删除已弃用的 meshes/link6.stl（含夹爪的完整网格）；新增 link6_trimmed.stl、adapter.stl

验证：
- URDF(自写 FK) vs MJCF(mujoco) 8 组随机位姿，12 个关键 link（含 5 个指尖）世界位置
  最大偏差 1.1e-6 m（远小于 1e-4；此前为 1.1e-2 m）
- 目检：离屏渲出"旧 link6.stl"与"新 link6_trimmed + adapter"，确认新模型无夹爪、可见连接件圆盘；
  "link6 + adapter + 手基座/拇指/食指"装配图确认手通过连接件挂在法兰前 17.5mm
- 查看器资源 HTTP 全 200（URDF 引用的 20 个网格）
- docs/viewer/index.html：手部映射的远端联动限位同步为 MJCF 值（thumb_ip 1.3282、dip 1.424），
  副标题/说明卡片注明模型来源与"无夹爪+连接件"

File: docs/viewer/robot.urdf (robot description, URDF)
Before this commit: robot piper_linkerhand_o6_left, 19 links, 18 joints
Links:
- link base_link: mass 1.02 -> None; geometry visual mesh filename=meshes/base_link.stl
- link lh_hand_base_link: mass 0.0672935238166485 -> None; geometry visual mesh filename=meshes/hand_base_link.stl
- link lh_index_distal: mass 0.00376951085886838 -> None; geometry visual mesh filename=meshes/index_distal.stl
- link lh_index_proximal: mass 0.00253174651934627 -> None; geometry visual mesh filename=meshes/index_proximal.stl
- link lh_middle_distal: mass 0.00376952789210256 -> None; geometry visual mesh filename=meshes/middle_distal.stl
- link lh_middle_proximal: mass 0.00253177375206983 -> None; geometry visual mesh filename=meshes/middle_proximal.stl
- link lh_pinky_distal: mass 0.00376948071276134 -> None; geometry visual mesh filename=meshes/pinky_distal.stl
- link lh_pinky_proximal: mass 0.00253185993162408 -> None; geometry visual mesh filename=meshes/pinky_proximal.stl
- link lh_ring_distal: mass 0.00376949588316609 -> None; geometry visual mesh filename=meshes/ring_distal.stl
- link lh_ring_proximal: mass 0.00253182223645066 -> None; geometry visual mesh filename=meshes/ring_proximal.stl
- link lh_thumb_distal: mass 0.00763332957284057 -> None; geometry visual mesh filename=meshes/thumb_distal.stl
- link lh_thumb_metacarpals: mass 0.0123381586619931 -> None; geometry visual mesh filename=meshes/thumb_metacarpals.stl
- link lh_thumb_metacarpals_base2: mass 0.00138588296544333 -> None; geometry visual mesh filename=meshes/thumb_metacarpals_base2.stl
- link link1: mass 0.71 -> None; geometry visual mesh filename=meshes/link1.stl
- link link2: mass 1.17 -> None; geometry visual mesh filename=meshes/link2.stl
- link link3: mass 0.5 -> None; geometry visual mesh filename=meshes/link3.stl
- link link4: mass 0.38 -> None; geometry visual mesh filename=meshes/link4.stl
- link link5: mass 0.383 -> None; geometry visual mesh filename=meshes/link5.stl
- link link6: mass 0.00699089613564366 -> None; geometry visual mesh filename=meshes/adapter.stl; visual mesh filename=meshes/link6_trimmed.stl
Joints:
- joint joint1: limit lower=-2.618 upper=2.168 effort=100 velocity=5 -> lower=-2.618 upper=2.618 effort=100 velocity=5; origin xyz=0 0 0.123 rpy=0 0 0 -> xyz=0 0 0.123 rpy=0 0 -1.5708
- joint joint2: origin xyz=0 0 0 rpy=1.5708 -0.1359 -3.1416 -> xyz=0 0 0 rpy=1.5708 8.00005e-12 -1.5708
- joint joint3: limit lower=-2.967 upper=0 effort=100 velocity=5 -> lower=-2.697 upper=0 effort=100 velocity=5; origin xyz=0.28503 0 0 rpy=0 0 -1.7939 -> xyz=0.28358 0.028726 0 rpy=0 0 0.10095
- joint joint4: limit lower=-1.745 upper=1.745 effort=100 velocity=5 -> lower=-1.832 upper=1.832 effort=100 velocity=5; origin xyz=-0.021984 -0.25075 0 rpy=1.5708 0 0 -> xyz=-0.24221 0.068514 0 rpy=-1.5708 7.13697e-07 1.3826
- joint joint5: origin xyz=0 0 0 rpy=-1.5708 0 0 -> xyz=0 0 0 rpy=1.5708 0 0
- joint joint6: limit lower=-2.0944 upper=2.0944 effort=100 velocity=3 -> lower=-3.14 upper=3.14 effort=100 velocity=5; origin xyz=8.8259E-05 -0.091 0 rpy=1.5708 0 0 -> xyz=0 0.091 0.0014165 rpy=1.57079 0 -3.14159
- joint lh_index_dip: limit lower=0 upper=1.43 effort=100 velocity=1 -> lower=0 upper=1.424 effort=100 velocity=5; mimic joint=lh_index_mcp_pitch multiplier=0.89 offset=0 -> (none)
- joint lh_index_mcp_pitch: limit lower=0 upper=1.60 effort=100 velocity=1 -> lower=0 upper=1.6 effort=100 velocity=5
- joint lh_middle_dip: limit lower=0 upper=1.43 effort=100 velocity=1 -> lower=0 upper=1.424 effort=100 velocity=5; mimic joint=lh_middle_mcp_pitch multiplier=0.89 offset=0 -> (none)
- joint lh_middle_mcp_pitch: limit lower=0 upper=1.60 effort=100 velocity=1 -> lower=0 upper=1.6 effort=100 velocity=5
- joint lh_pinky_dip: limit lower=0 upper=1.43 effort=100 velocity=1 -> lower=0 upper=1.424 effort=100 velocity=5; mimic joint=lh_pinky_mcp_pitch multiplier=0.89 offset=0 -> (none)
- joint lh_pinky_mcp_pitch: limit lower=0 upper=1.60 effort=100 velocity=1 -> lower=0 upper=1.6 effort=100 velocity=5; origin xyz=0.0024758 0.028372 0.092741 rpy=-0.087266 0 0 -> xyz=0.0024758 0.028372 0.092741 rpy=-0.0872661 0 0
- joint lh_ring_dip: limit lower=0 upper=1.43 effort=100 velocity=1 -> lower=0 upper=1.424 effort=100 velocity=5; mimic joint=lh_ring_mcp_pitch multiplier=0.89 offset=0 -> (none)
- joint lh_ring_mcp_pitch: limit lower=0 upper=1.60 effort=100 velocity=1 -> lower=0 upper=1.6 effort=100 velocity=5
- joint lh_thumb_cmc_pitch: limit lower=0 upper=0.58 effort=100 velocity=1 -> lower=0 upper=0.58 effort=100 velocity=5; origin xyz=0.0061649 -0.010678 -0.004891 rpy=0 -1.1529 2.0944 -> xyz=0.0061649 -0.010678 -0.004891 rpy=2.97362e-06 -1.1529 2.0944
- joint lh_thumb_cmc_yaw: limit lower=0 upper=1.3 effort=100 velocity=1 -> lower=0 upper=1.3 effort=100 velocity=5
- joint lh_thumb_ip: limit lower=0 upper=1.08 effort=100 velocity=1 -> lower=0 upper=1.3282 effort=100 velocity=5; mimic joint=lh_thumb_cmc_pitch multiplier=2.29 offset=0 -> (none)
